Commit message: Refactor arm.urdf to improve link and joint naming conventions for clarity. Update ServoControllerNode to enhance servo initialization logging and error handling.

File: arm_controller/description/arm.urdf (robot description, URDF)
Before this commit: robot two_joint_arm, 3 links, 2 joints
Links:
- removed link base_link
- removed link link1
- removed link link2
- added link base; visual cylinder length=.5 radius=2
- added link elbow; visual box size=1 1 5
- added link shoulder; visual box size=1 1 1
Joints:
- removed joint joint2
- added joint joint0: type revolute, parent base, child shoulder, origin xyz=0 0 1 rpy=0 0 0, axis 0 0 1, limit lower=-3.14 upper=3.14 effort=100 velocity=1
- joint joint1: axis 0 0 1 -> 1 0 0; child link1 -> elbow; origin xyz=0 0 1 rpy=0 0 0 -> xyz=1 0 0 rpy=0 0 0; parent base_link -> shoulder

Commit message: Enhance arm.urdf by adding inertial properties, collision geometries, and a new wrist link and joint. Update existing links with origins and adjust dimensions for better accuracy in the robot model.

File: arm_controller/description/arm.urdf (robot description, URDF)
Before this commit: robot two_joint_arm, 3 links, 2 joints
Links:
- added link wrist, mass 0.5; collision box size=0.5 0.5 2; visual box size=0.5 0.5 2
- link base: geometry collision cylinder length=.5 radius=2; visual cylinder length=.5 radius=2
- link elbow: mass None -> 1.0; geometry collision box size=1 1 5; visual box size=1 1 3
- link shoulder: mass None -> 1.0; geometry collision box size=1 1 1; visual box size=1 1 1
Joints:
- added joint joint2: type revolute, parent elbow, child wrist, origin xyz=0 0 5 rpy=0 0 0, axis 1 0 0, limit lower=-3.14 upper=3.14 effort=50 velocity=1
