Commit message: back to using only 2 joints

File: servo42c_controller/description/arm.urdf (robot description, URDF)
Before this commit: robot two_joint_arm, 4 links, 3 joints
Links:
- removed link wrist
Joints:
- removed joint joint0
- joint joint1: axis 1 0 0 -> 0 0 1; child elbow -> shoulder; limit lower=-3.14 upper=3.14 effort=100 velocity=1 -> lower=-3.14 upper=3.14 effort=100 velocity=100; origin xyz=1 0 0 rpy=0 0 0 -> xyz=0 0 1 rpy=0 0 0; parent shoulder -> base
- joint joint2: child wrist -> elbow; limit lower=-3.14 upper=3.14 effort=50 velocity=1 -> lower=-3.14 upper=3.14 effort=100 velocity=100; origin xyz=0 0 5 rpy=0 0 0 -> xyz=1 0 0 rpy=0 0 0; parent elbow -> shoulder
